File: Z80_miniCore.kicad_pcb (KiCad board)
At the start: 2 copper layers, 92.5 x 80 mm, 40 parts, among them J1 ICSP, J2 UART, J3 I2C, J5 MicroSD, J7 USB_B_Mini, SW1 ON|OFF, SW2 Z80_RESET, SW3 CUSTOM, U1 Z84C00/PLCC, U2 PIC1-MMU, U3 28C256, U4 74HC138, U7 IS62C256AL, Y1 CANNED-DIP8, Y2 Crystal

Commit message: finish routing.
Parts:
- moved Y1 0.31 mm to (124.5, 84.8)
Connections:
- U4 pad 5: /RFSH -> GND
Routing:
- net /D2: track 0.00 -> 117.2 mm, vias 0 -> 7
- net /D7: track 0.00 -> 106.7 mm, vias 0 -> 10
- net /D1: track 0.00 -> 100.2 mm, vias 0 -> 5
- net /D3: track 0.00 -> 99.9 mm, vias 0 -> 8
- net Net-(J7-VBUS): track 0.00 -> 96.5 mm
- net /D0: track 0.00 -> 96.4 mm, vias 0 -> 5
- net /D4: track 0.00 -> 93.5 mm, vias 0 -> 6
- net /RD: track 0.00 -> 92.8 mm, vias 0 -> 5
- net /INT: track 0.00 -> 92.7 mm, vias 0 -> 5
- net /WR: track 0.00 -> 90.8 mm, vias 0 -> 8
- net /HALT: track 0.00 -> 90.6 mm, vias 0 -> 8
- net /RESET: track 0.00 -> 88.2 mm, vias 0 -> 9
- net /MREQ: track 0.00 -> 87.4 mm, vias 0 -> 3
- net /A0: track 0.00 -> 86.6 mm, vias 0 -> 5
- net /D5: track 0.00 -> 85.7 mm, vias 0 -> 7
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- added copper zone on B.Cu, net GND
- added copper zone on F.Cu, net VCC
Other:
- board text added: "Z80-miniCore-32K Rev.4 @ 06.08.26 Author: @thetrung Made With KiCAD"
