File: Z80_miniCore.kicad_pcb (KiCad board)
At the start: 2 copper layers, 92.5 x 80 mm, 40 parts, among them J1 ICSP, J2 UART, J3 I2C, J5 MicroSD, J7 USB_B_Mini, SW1 ON|OFF, SW2 Z80_RESET, SW3 CUSTOM, U1 Z84C00/PLCC, U2 PIC1-MMU, U3 28C256, U4 74HC138, U7 IS62C256AL, Y1 CANNED-DIP8, Y2 Crystal

Commit message: Replace 8x10K_R w/ 1xRN8. Refine footprints.
Parts:
- removed R10, R11, R12, R4, R5, R6, R7, R9: 10K, Resistor_THT:R_Axial_DIN0207_L6.3mm_D2.5mm_P10.16mm_Horizontal
- added RN1: R_Network08, Resistor_THT:R_Array_SIP9, F.Cu at (138.2, 103.0)
- C8: footprint Capacitor_THT:C_Disc_D3.4mm_W2.1mm_P2.50mm -> Capacitor_THT:C_Radial_D4.0mm_H5.0mm_P1.50mm
- C9: value 100uF -> 10uF
- J5: footprint Connector_PinSocket_2.54mm:PinSocket_1x06_P2.54mm_Vertical -> Connector_PinHeader_2.54mm:PinHeader_1x06_P2.54mm_Vertical
- R13: value 4k7 -> 10K
- R14: value 330 -> 1K
- moved C8 43.6 mm to (193.5, 89.2), turned to 90 degrees
- moved R8 42.4 mm to (112.1, 102.0), turned to 0 degrees
- moved J5 27.0 mm to (198.0, 77.0), turned to 0 degrees
- moved J1 3.50 mm to (185.4, 39.5)
- moved SW1 2.92 mm to (120.0, 93.5)
Routing:
- net /RESET: track 88.2 -> 104.9 mm, vias 9 -> 6
- net /SCK: track 59.2 -> 43.5 mm
- net /NMI: track 7.78 -> 22.9 mm, vias 1 -> 2
- net /INT: track 92.7 -> 85.9 mm, vias 5 -> 7
- net /IORQ: track 62.1 -> 68.8 mm, vias 3 -> 6
- net /CS: track 45.7 -> 40.6 mm
- net /MOSI: track 52.6 -> 47.5 mm, vias 2 -> 1
- net /PGC: track 23.4 -> 26.9 mm, vias 0 -> 1
- net /PGD: track 27.2 -> 30.7 mm
- net Net-(J7-VBUS): track 96.5 -> 93.5 mm
- net /MREQ: track 87.4 -> 85.1 mm
- net /BUSREQ: track 17.4 -> 19.5 mm, vias 0 -> 1
- net /WAIT: track 5.96 -> 7.78 mm
- net /MISO: track 45.1 -> 46.6 mm, vias 5 -> 1
- net /WR: track 90.8 -> 91.9 mm
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Other:
- board text added: "+"
- board text added: "CS"
- board text added: "GND"
- board text added: "ISO"
- board text added: "OSI"
- board text added: "RX"
- board text added: "SCK"
- board text added: "TX"
- board text added: "VCC"
